File: hackpad/hackpad.kicad_sch (KiCad schematic)
At the start: 0 parts

Commit message: update the PCB file
Parts:
- added SW1, SW2, SW3, SW4: SW_Push, Button_Switch_Keyboard:SW_Cherry_MX_1.00u_PCB, symbol Switch:SW_Push
- added U1: MOUDLE-SEEEDUINO-XIAO, footprints:XIAO-Generic-Hybrid-14P-2.54-21X17.8MM, symbol XIAO_RP2040:MOUDLE-SEEEDUINO-XIAO
- added U2: ER_OLEDM0.91_1x-I2C, Display:ER_OLEDM0.91_1x-I2C, symbol Display_Graphic:ER_OLEDM0.91_1x-I2C
Connections:
- new net: SW1.1, U1.1 (PA02_A0_D0)
- new net: SW2.1, U1.2 (PA4_A1_D1)
- new net: SW3.1, U1.3 (PA10_A2_D2)
- new net: SW4.1, U1.4 (PA11_A3_D3)
- new net: U1.5 (PA8_A4_D4_SDA), U2.4 (SDA)
- new net: U1.6 (PA9_A5_D5_SCL), U2.3 (SCL)
- new net GND: SW1.2, SW2.2, SW3.2, SW4.2, U1.13 (GND), U2.1 (GND)
- new net VDD: U1.12 (3V3), U2.2 (VCC)
